Commit message: First Commit

File: models/urdf/ROS_BOT_1.xacro (robot description, xacro)
@@ -104,4 +104,11 @@
   </collision>
 </link>
+<link name="camera">
+</link>
+<joint name="camera_joint" type="fixed">
+  <origin xyz="0.0 0.0 0.1" rpy="0 0 0"/>
+  <parent link="base_link"/>
+  <child link="camera"/>
+</joint>
 <joint name="right_wheel_joint" type="continuous">
   <origin xyz="-0.08 -0.06 0.03" rpy="0 0 0"/>
